Commit message: Added inertia

File: urdf/vehicle.xacro (robot description, xacro)
@@ -24,7 +24,7 @@
 	<link name="wheel_rear_right_link">
 		<intertial>
-			<origin xyz="0 0 0" rpy="0 0 0"/>
-			<mass value="0.0"/>
-			<inertia ixx="0.0" ixy="0.0" ixz="0.0" iyy="0.0" iyz="0.0" izz="0.0"/>
+			<origin xyz="0.0 0.0 0.0" rpy="0.0 0.0 0.0"/>
+			<mass value="1.0"/>
+			<inertia ixx="${(1/12)*(3*0.15*0.15+0.1*0.1)}" ixy="0.0" ixz="0.0" iyy="${(1/12)*(3*0.15*0.15+0.1*0.1)}" iyz="0.0" izz="${(1/2)*(0.15*0.15)}"/>
 		</intertial>
 		<visual name="">
@@ -53,7 +53,7 @@
 	<link name="wheel_rear_left_link">
 		<intertial>
-			<origin xyz="0 0 0" rpy="0 0 0"/>
-			<mass value="0.0"/>
-			<inertia ixx="0.0" ixy="0.0" ixz="0.0" iyy="0.0" iyz="0.0" izz="0.0"/>
+			<origin xyz="0.0 0.0 0.0" rpy="0.0 0.0 0.0"/>
+			<mass value="1.0"/>
+			<inertia ixx="${(1/12)*(3*0.15*0.15+0.1*0.1)}" ixy="0.0" ixz="0.0" iyy="${(1/12)*(3*0.15*0.15+0.1*0.1)}" iyz="0.0" izz="${(1/2)*(0.15*0.15)}"/>
 		</intertial>
 		<visual name="">
@@ -82,7 +82,7 @@
 	<link name="wheel_front_right_link">
 		<intertial>
-			<origin xyz="0 0 0" rpy="0 0 0"/>
-			<mass value="0.0"/>
-			<inertia ixx="0.0" ixy="0.0" ixz="0.0" iyy="0.0" iyz="0.0" izz="0.0"/>
+			<origin xyz="0.0 0.0 0.0" rpy="0.0 0.0 0.0"/>
+			<mass value="1.0"/>
+			<inertia ixx="${(1/12)*(3*0.15*0.15+0.1*0.1)}" ixy="0.0" ixz="0.0" iyy="${(1/12)*(3*0.15*0.15+0.1*0.1)}" iyz="0.0" izz="${(1/2)*(0.15*0.15)}"/>
 		</intertial>
 		<visual name="">
@@ -111,7 +111,7 @@
 	<link name="wheel_front_left_link">
 		<intertial>
-			<origin xyz="0 0 0" rpy="0 0 0"/>
-			<mass value="0.0"/>
-			<inertia ixx="0.0" ixy="0.0" ixz="0.0" iyy="0.0" iyz="0.0" izz="0.0"/>
+			<origin xyz="0.0 0.0 0.0" rpy="0.0 0.0 0.0"/>
+			<mass value="1.0"/>
+			<inertia ixx="${(1/12)*(3*0.15*0.15+0.1*0.1)}" ixy="0.0" ixz="0.0" iyy="${(1/12)*(3*0.15*0.15+0.1*0.1)}" iyz="0.0" izz="${(1/2)*(0.15*0.15)}"/>
 		</intertial>
 		<visual name="">
