Commit message: abstraction

File: urdf/vehicle.urdf.xacro (robot description, xacro)
@@ -22,6 +22,6 @@
                 </visual>
         </link>
-	<link name="wheel_rear_right_link">
-		<!--
+	<xacro:property name="side1" value="rear_right"/>
+	<link name="wheel_${side1}_link">
 		<intertial>
 			<origin xyz="0.0 0.0 0.0" rpy="0.0 0.0 0.0"/>
@@ -29,5 +29,4 @@
 			<inertia ixx="${(1/12)*(3*0.15*0.15+0.1*0.1)}" ixy="0.0" ixz="0.0" iyy="${(1/12)*(3*0.15*0.15+0.1*0.1)}" iyz="0.0" izz="${(1/2)*(0.15*0.15)}"/>
 		</intertial>
-		-->
 		<visual name="">
 			<origin xyz="0.0 0.0 0.0" rpy="0.0 0.0 0.0"/>
@@ -47,12 +46,12 @@
 		</collision>
 	</link>
-	<joint name="wheel_rear_right_joint" type="continuous">
-		<origin xyz="0.250 0.40 0.0" rpy="1.57 0.0 0.0"/>
+	<joint name="wheel_${side1}_joint" type="continuous">
+		<origin xyz="-0.250 -0.40 0.0" rpy="1.57 0.0 0.0"/>
 		<parent link="base_link"/>
-		<child link="wheel_rear_right_link"/>
+		<child link="wheel_${side1}_link"/>
 		<axis xyz="0.0 0.0 1.0"/>
 	</joint>
-	<link name="wheel_rear_left_link">
-		<!--
+	<xacro:property name="side2" value="rear_left"/>
+	<link name="wheel_${side2}_link">
 		<intertial>
 			<origin xyz="0.0 0.0 0.0" rpy="0.0 0.0 0.0"/>
@@ -60,5 +59,4 @@
 			<inertia ixx="${(1/12)*(3*0.15*0.15+0.1*0.1)}" ixy="0.0" ixz="0.0" iyy="${(1/12)*(3*0.15*0.15+0.1*0.1)}" iyz="0.0" izz="${(1/2)*(0.15*0.15)}"/>
 		</intertial>
-		-->
 		<visual name="">
 			<origin xyz="0.0 0.0 0.0" rpy="0.0 0.0 0.0"/>
@@ -78,12 +76,12 @@
 		</collision>
 	</link>
-	<joint name="wheel_rear_left_joint" type="continuous">
-		<origin xyz="0.250 -0.40 0.0" rpy="1.57 0.0 0.0"/>
+	<joint name="wheel_${side2}_joint" type="continuous">
+		<origin xyz="-0.250 0.40 0.0" rpy="1.57 0.0 0.0"/>
 		<parent link="base_link"/>
-		<child link="wheel_rear_left_link"/>
+		<child link="wheel_${side2}_link"/>
 		<axis xyz="0.0 0.0 1.0"/>
 	</joint>
-	<link name="wheel_front_right_link">
-		<!--
+	<xacro:property name="side3" value="front_right"/>
+	<link name="wheel_${side3}_link">
 		<intertial>
 			<origin xyz="0.0 0.0 0.0" rpy="0.0 0.0 0.0"/>
@@ -91,5 +89,4 @@
 			<inertia ixx="${(1/12)*(3*0.15*0.15+0.1*0.1)}" ixy="0.0" ixz="0.0" iyy="${(1/12)*(3*0.15*0.15+0.1*0.1)}" iyz="0.0" izz="${(1/2)*(0.15*0.15)}"/>
 		</intertial>
-		-->
 		<visual name="">
 			<origin xyz="0.0 0.0 0.0" rpy="0.0 0.0 0.0"/>
@@ -109,12 +106,12 @@
 		</collision>
 	</link>
-	<joint name="wheel_front_right_joint" type="continuous">
-		<origin xyz="-0.250 0.40 0.0" rpy="1.57 0.0 0.0"/>
+	<joint name="wheel_${side3}_joint" type="continuous">
+		<origin xyz="0.250 -0.40 0.0" rpy="1.57 0.0 0.0"/>
 		<parent link="base_link"/>
-		<child link="wheel_front_right_link"/>
+		<child link="wheel_${side3}_link"/>
 		<axis xyz="0.0 0.0 1.0"/>
 	</joint>
-	<link name="wheel_front_left_link">
-		<!--
+	<xacro:property name="side4" value="front_left"/>
+	<link name="wheel_${side4}_link">
 		<intertial>
 			<origin xyz="0.0 0.0 0.0" rpy="0.0 0.0 0.0"/>
@@ -122,5 +119,4 @@
 			<inertia ixx="${(1/12)*(3*0.15*0.15+0.1*0.1)}" ixy="0.0" ixz="0.0" iyy="${(1/12)*(3*0.15*0.15+0.1*0.1)}" iyz="0.0" izz="${(1/2)*(0.15*0.15)}"/>
 		</intertial>
-		-->
 		<visual name="">
 			<origin xyz="0.0 0.0 0.0" rpy="0.0 0.0 0.0"/>
@@ -140,8 +136,8 @@
 		</collision>
 	</link>
-	<joint name="wheel_front_left_joint" type="continuous">
-		<origin xyz="-0.250 -0.40 0.0" rpy="1.57 0.0 0.0"/>
+	<joint name="wheel_${side4}_joint" type="continuous">
+		<origin xyz="0.250 0.40 0.0" rpy="1.57 0.0 0.0"/>
 		<parent link="base_link"/>
-		<child link="wheel_front_left_link"/>
+		<child link="wheel_${side4}_link"/>
 		<axis xyz="0.0 0.0 1.0"/>
 	</joint>
